File: Loom/New BSPD/power.kicad_sch (KiCad schematic)
At the start: 13 parts, among them J4 Screw_Terminal_01x02, U1 4011, U10 LM2901, U11 4012, U16 L7805, U2 4011, U3 4011, U4 4011, U5 4011, U6 4011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

Commit message: Complete Schematic, Footprint Assignment, Start PCB Design
Parts:
- J4: footprint (none) -> TerminalBlock:TerminalBlock_bornier-2_P5.08mm
- U1, U10, U11, U2, U3, U4, U5, U6, U7, U8, U9: footprint (none) -> Package_DIP:DIP-14_W7.62mm_Socket
- U16: footprint (none) -> Package_TO_SOT_THT:TO-220-3_Horizontal_TabDown
Changed lines of the file:
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@@
       (effects (font (size 1.27 1.27)) (justify left))
     )
-    (property "Footprint" "" (at 109.22 110.49 0)
+    (property "Footprint" "Package_DIP:DIP-14_W7.62mm_Socket" (at 109.22 110.49 0)
       (effects (font (size 1.27 1.27)) hide)
     )
@@
       (effects (font (size 1.27 1.27)) (justify left))
     )
-    (property "Footprint" "" (at 80.01 113.03 0)
+    (property "Footprint" "Package_DIP:DIP-14_W7.62mm_Socket" (at 80.01 113.03 0)
       (effects (font (size 1.27 1.27)) hide)
     )
@@
       (effects (font (size 1.27 1.27)) (justify left))
     )
-    (property "Footprint" "" (at 44.45 113.03 0)
+    (property "Footprint" "Package_DIP:DIP-14_W7.62mm_Socket" (at 44.45 113.03 0)
       (effects (font (size 1.27 1.27)) hide)
     )
@@
       (effects (font (size 1.27 1.27)))
     )
-    (property "Footprint" "" (at 42.545 33.02 0)
+    (property "Footprint" "Package_TO_SOT_THT:TO-220-3_Horizontal_TabDown" (at 42.545 33.02 0)
       (effects (font (size 1.27 1.27) italic) (justify left) hide)
     )
@@
       (effects (font (size 1.27 1.27)) (justify left))
     )
-    (property "Footprint" "" (at 73.66 30.48 0)
+    (property "Footprint" "TerminalBlock:TerminalBlock_bornier-2_P5.08mm" (at 73.66 30.48 0)
       (effects (font (size 1.27 1.27)) hide)
     )
@@
       (effects (font (size 1.27 1.27)) (justify left))
     )
-    (property "Footprint" "" (at 26.67 113.03 0)
+    (property "Footprint" "Package_DIP:DIP-14_W7.62mm_Socket" (at 26.67 113.03 0)
       (effects (font (size 1.27 1.27)) hide)
     )
@@
       (effects (font (size 1.27 1.27)) (justify left))
     )
-    (property "Footprint" "" (at 71.12 113.03 0)
+    (property "Footprint" "Package_DIP:DIP-14_W7.62mm_Socket" (at 71.12 113.03 0)
       (effects (font (size 1.27 1.27)) hide)
     )
@@
       (effects (font (size 1.27 1.27)) (justify left))
     )
-    (property "Footprint" "" (at 53.34 113.03 0)
+    (property "Footprint" "Package_DIP:DIP-14_W7.62mm_Socket" (at 53.34 113.03 0)
       (effects (font (size 1.27 1.27)) hide)
     )
@@
       (effects (font (size 1.27 1.27)) (justify left))
     )
-    (property "Footprint" "" (at 99.06 110.49 0)
+    (property "Footprint" "Package_DIP:DIP-14_W7.62mm_Socket" (at 99.06 110.49 0)
       (effects (font (size 1.27 1.27)) hide)
     )
@@
       (effects (font (size 1.27 1.27)) (justify left))
     )
-    (property "Footprint" "" (at 35.56 113.03 0)
+    (property "Footprint" "Package_DIP:DIP-14_W7.62mm_Socket" (at 35.56 113.03 0)
       (effects (font (size 1.27 1.27)) hide)
     )
@@
       (effects (font (size 1.27 1.27)) (justify left))
     )
-    (property "Footprint" "" (at 62.23 113.03 0)
+    (property "Footprint" "Package_DIP:DIP-14_W7.62mm_Socket" (at 62.23 113.03 0)
       (effects (font (size 1.27 1.27)) hide)
     )
@@
       (effects (font (size 1.27 1.27)) (justify left))
     )
-    (property "Footprint" "" (at 118.11 113.03 0)
+    (property "Footprint" "Package_DIP:DIP-14_W7.62mm_Socket" (at 118.11 113.03 0)
       (effects (font (size 1.27 1.27)) hide)
     )
@@
       (effects (font (size 1.27 1.27)) (justify left))
     )
-    (property "Footprint" "" (at 88.9 113.03 0)
-      (effects (font (size 1.27 1.27)) hide)
-    )
+    (property "Footprint" "Package_DIP:DIP-14_W7.62mm_Socket" (at 88.9 113.03 0)
+      (effects (font (size 1.27 1.27)) hide)
+    )
