File: Loom/New BSPD/power.kicad_sch (KiCad schematic)
At the start: 13 parts, among them J4 Screw_Terminal_01x02, U1 4011, U10 LM2901, U11 4012, U16 L7805, U2 4011, U3 4011, U4 4011, U5 4011, U6 4011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

Commit message: Change BSPD Power connector
Parts:
- J4: footprint TerminalBlock:TerminalBlock_bornier-2_P5.08mm -> BSPD_footprints:ATF13-2P-BM03
Changed lines of the file:
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@@
       (effects (font (size 1.27 1.27)) (justify left))
     )
-    (property "Footprint" "TerminalBlock:TerminalBlock_bornier-2_P5.08mm" (at 73.66 30.48 0)
+    (property "Footprint" "BSPD_footprints:ATF13-2P-BM03" (at 73.66 30.48 0)
       (effects (font (size 1.27 1.27)) hide)
     )
