File: Loom/New BSPD/reset.kicad_sch (KiCad schematic)
At the start: 4 parts, among them U10 LM2901

Commit message: Complete Schematic, Footprint Assignment, Start PCB Design
Parts:
- C1: value C -> 100n; footprint (none) -> Capacitor_THT:C_Disc_D5.0mm_W2.5mm_P5.00mm
- R8: value R -> 1M; footprint (none) -> Resistor_THT:R_Axial_DIN0207_L6.3mm_D2.5mm_P7.62mm_Horizontal
- RV5: footprint (none) -> Potentiometer_THT:Potentiometer_Bourns_3296Y_Vertical
- U10: footprint (none) -> Package_DIP:DIP-14_W7.62mm_Socket
Changed lines of the file:
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@@
       (effects (font (size 1.27 1.27)))
     )
-    (property "Footprint" "" (at 114.3 26.67 0)
+    (property "Footprint" "Package_DIP:DIP-14_W7.62mm_Socket" (at 114.3 26.67 0)
       (effects (font (size 1.27 1.27)) hide)
     )
@@
       (effects (font (size 1.27 1.27)))
     )
-    (property "Value" "C" (at 90.17 38.1 90)
+    (property "Value" "100n" (at 90.17 38.1 90)
       (effects (font (size 1.27 1.27)))
     )
-    (property "Footprint" "" (at 93.98 42.2148 0)
+    (property "Footprint" "Capacitor_THT:C_Disc_D5.0mm_W2.5mm_P5.00mm" (at 93.98 42.2148 0)
       (effects (font (size 1.27 1.27)) hide)
     )
-    (property "Datasheet" "~" (at 90.17 43.18 0)
+    (property "Datasheet" "MULTICOMP PRO MCFYU6104Z6" (at 90.17 43.18 0)
       (effects (font (size 1.27 1.27)) hide)
     )
@@
       (effects (font (size 1.27 1.27)) (justify right))
     )
-    (property "Footprint" "" (at 90.17 26.67 0)
+    (property "Footprint" "Potentiometer_THT:Potentiometer_Bourns_3296Y_Vertical" (at 90.17 26.67 0)
       (effects (font (size 1.27 1.27)) hide)
     )
@@
       (effects (font (size 1.27 1.27)))
     )
-    (property "Value" "R" (at 100.33 39.37 90)
+    (property "Value" "1M" (at 100.33 39.37 90)
       (effects (font (size 1.27 1.27)))
     )
-    (property "Footprint" "" (at 100.33 44.958 90)
+    (property "Footprint" "Resistor_THT:R_Axial_DIN0207_L6.3mm_D2.5mm_P7.62mm_Horizontal" (at 100.33 44.958 90)
       (effects (font (size 1.27 1.27)) hide)
     )
