File: Loom/Can Pcb/CAN_PCB.kicad_sch (KiCad schematic)
At the start: 28 parts, among them J1 Conn_01x02, J12 Conn_01x03, J15 Conn_01x03, J16 Conn_01x03, J2 Conn_01x05_Pin, J4 Conn_01x02, J5 Conn_01x03, U2 MCP2551-I-P, U4 TL780-05KCS, Y1 Crystal

Commit message: Added various files
Parts:
- removed C3, C4, C5, C6: C, Capacitor_THT:C_Disc_D4.7mm_W2.5mm_P5.00mm, symbol Device:C
- removed J1: Conn_01x02, Footprints:ATF13-2P-BM03, symbol Connector_Generic:Conn_01x02
- added J3: Screw_Terminal_01x02, TerminalBlock:TerminalBlock_bornier-2_P5.08mm, symbol Connector:Screw_Terminal_01x02
Connections:
- net +12V: now also J3.2 (Pin_2)
- net GND: now also J3.1 (Pin_1)
Other:
- note removed: "+12V"
